File: VERTECS_CCB/VERTECS_CCB_A.kicad_pcb (KiCad board)
At the start: 4 copper layers, 90 x 74 mm, 219 parts, among them IC1 AD7490BCPZ, IC2 FSUSB42UMX, IC3 FT232HQ, IC4 LTC4361IDC-2#TRMPBF, IC5 LTC4361IDC-2#TRMPBF, IC6 LTC4361IDC-2#TRMPBF, J1 DF14-30P-1.25H_35_, J10 1-1734248-5, J11 2137160001, J12 2137160001, J13 55460-0272, J14 55460-0272, J15 55460-0272, J16 55460-0272, J17 55460-0272, J2 DF14-4P-1.25H_35_, J3 DF14-7P-1.25H_35_, J4 Conn_01x03, J5 ER8-20S-0.8SV-5H, J6 Conn_01x02, J7 Conn_01x02, J9 1-1734248-5, Q1 SSM6K514NU,LF, Q2 SSM6K514NU,LF, Q3 SSM6K514NU,LF, Q4 SSM6K514NU,LF, Q5 SSM6K514NU,LF, Q6 SSM6K514NU,LF, Q7 SSM6K514NU,LF, Q8 SSM6K514NU,LF, U1 74LVC1G07SE-7, U10 LTC4380HDD-1-PBF, U11 SSM6K403TU,LF, U12 DTC144EET1G, U13 SSM6K403TU,LF, U14 DTC144EET1G, U15 DTC144EET1G, U16 TLP293, U2 2337822-2, U3 USB2514B-I/M2, U4 AP22653W6-7, U5 SSM6K403TU,LF, U6 DTC144EET1G, U7 LTC4380HDD-1-PBF, U8 LTC4380HDD-1-PBF, U9 LTC4380HDD-1-PBF, Y1 24MHz, Y2 12MHz

Commit message: Update to v1.4
Parts:
- removed C63, C64, C65, C66, C67, C68, C69, C70: 15pF N.F., Resistor_SMD:R_0402_1005Metric
- removed R71, R72, R73, R74, R75, R76, R77, R78: 49R9 N.F., Resistor_SMD:R_0402_1005Metric
- FID1, FID2: value Fiducial_1mm_Mask2mm -> Fiducial
- moved FID1 3.70 mm to (107.8, 120.8)
- moved G*** 3.05 mm to (160.4, 89.6)
Routing:
- net /CM4 GPIO/+3.3v: track 269.3 -> 233.6 mm, vias 7 -> 8
- net /+5v_RPI: track 135.3 -> 105.3 mm
- net GND: track 500.1 -> 483.5 mm, vias 184 -> 180
- net /CM4 GPIO/TRD0_N: track 35.6 -> 31.1 mm, vias 1 -> 0
- net Net-(Module1A-PI_nLED_Activity): track 50.6 -> 46.1 mm
- net /CM4 GPIO/TRD0_P: track 37.6 -> 33.3 mm
- net /CM4 GPIO/TRD3_P: track 15.5 -> 11.2 mm
- net /CM4 GPIO/TRD2_P: track 24.0 -> 19.8 mm
- net /CM4 GPIO/TRD2_N: track 20.8 -> 16.6 mm, vias 1 -> 0
- net /CM4 GPIO/TRD1_N: track 27.1 -> 22.9 mm, vias 1 -> 0
- net /CM4 GPIO/TRD1_P: track 28.1 -> 23.8 mm
- net /CM4 GPIO/TRD3_N: track 14.7 -> 10.6 mm, vias 1 -> 0
- net /CM4 GPIO/ETH_LEDG: track 44.6 -> 41.9 mm
- net /CM4 GPIO/CE0: track 33.8 -> 32.4 mm
- net /OBC-CCB_PWR_ON_DIO: track 45.4 -> 46.7 mm
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Other:
- board text added: "GND"
- board text added: "RX"
- board text added: "TX"
- board text added: "VERTECS CCB V1.4"
- board text removed: "VERTECS CCB-A Engineering Model V1.3"
