File: VERTECS_CCB/ethernet.kicad_sch (KiCad schematic)
At the start: 28 parts, among them J1 2337822-2, J5 ER8-20S-0.8SV-5H

Commit message: Update to v1.4
Parts:
- removed C63, C64, C65, C66, C67, C68, C69, C70: 15pF N.F., Resistor_SMD:R_0402_1005Metric, symbol Device:C
- removed R71, R72, R73, R74, R75, R76, R77, R78: 49R9 N.F., Resistor_SMD:R_0402_1005Metric, symbol Device:R
Other:
- moved on the sheet: C1, C2, J1, R1, R2, R3, R4
