File: VERTECS_CCB/usb_hub.kicad_sch (KiCad schematic)
At the start: 34 parts, among them IC1 FSUSB42UMX, J11 2137160001, J12 2137160001, U1 USB2514B-I/M2, U2 AP22653W6-7, Y1 24MHz

Commit message: Update to v1.4
Parts:
- R19, R20, R23, R24: Manufacturer_Part_Number RK73B1ETTP563J -> RK73H1ETTP5602F
Changed lines of the file:
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@@
   (title_block
     (title "VERTECS CCB - USB Hub Implementation")
-    (date "2024-05-28")
-    (rev "1.3")
+    (date "2024-09-11")
+    (rev "1.4")
     (company "Kyushu Institute of Technology")
     (comment 1 "See CM4 IO board datasheet for reference")
@@
       (effects (font (size 1.27 1.27)) hide)
     )
-    (property "Manufacturer_Part_Number" "RK73B1ETTP563J" (at 276.86 45.72 0)
+    (property "Manufacturer_Part_Number" "RK73H1ETTP5602F" (at 276.86 45.72 0)
       (effects (font (size 1.27 1.27)) hide)
     )
@@
       (effects (font (size 1.27 1.27)) hide)
     )
-    (property "Manufacturer_Part_Number" "RK73B1ETTP563J" (at 213.36 93.98 0)
+    (property "Manufacturer_Part_Number" "RK73H1ETTP5602F" (at 213.36 93.98 0)
       (effects (font (size 1.27 1.27)) hide)
     )
@@
       (effects (font (size 1.27 1.27)) hide)
     )
-    (property "Manufacturer_Part_Number" "RK73B1ETTP563J" (at 213.36 45.72 0)
+    (property "Manufacturer_Part_Number" "RK73H1ETTP5602F" (at 213.36 45.72 0)
       (effects (font (size 1.27 1.27)) hide)
     )
@@
       (effects (font (size 1.27 1.27)) hide)
     )
-    (property "Manufacturer_Part_Number" "RK73B1ETTP563J" (at 276.86 93.98 0)
-      (effects (font (size 1.27 1.27)) hide)
-    )
+    (property "Manufacturer_Part_Number" "RK73H1ETTP5602F" (at 276.86 93.98 0)
+      (effects (font (size 1.27 1.27)) hide)
+    )
